File: V1/relay-24v-8ch-8a-v1.kicad_sch (KiCad schematic)
At the start: 44 parts, among them J1 DB141V-2.54-6P, J2 DB141V-2.54-6P

Commit message: Update relay-24v-8ch-8a-v1.kicad_sch
Parts:
- gave numbers to parts that had none: 42
