File: V1/relay-24v-8ch-8a-v1.kicad_pcb (KiCad board)
At the start: 2 copper layers, 98 x 67.8 mm, 44 parts, among them J1 DB141V-2.54-6P, J2 DB141V-2.54-6P, J3 DB142V-5.08-8P, J4 DB142V-5.08-8P, K1 G5Q-1A4-DC24V, K2 G5Q-1A4-DC24V, K3 G5Q-1A4-DC24V, K4 G5Q-1A4-DC24V, K5 G5Q-1A4-DC24V, K6 G5Q-1A4-DC24V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

Commit message: Prefab checks
Parts:
- added J5: DB142V-5.08-4P, Tales:TerminalBlock_Dibo_DB142V-5.08-4P_1x04_P5.08mm_Vertical, F.Cu at (177.0, 122.6)
- added J6: DB142V-5.08-4P, Tales:TerminalBlock_Dibo_DB142V-5.08-4P_1x04_P5.08mm_Vertical, F.Cu at (201.0, 122.6)
- D1, D11, D13, D15, D3, D5, D7, D9: value GREEN -> EMERALD
- J3, J4: value DB142V-5.08-8P -> DB142V-5.08-4P; footprint Tales:TerminalBlock_Dibo_DB142V-5.08-8P_1x08_P5.08mm_Vertical -> Tales:TerminalBlock_Dibo_DB142V-5.08-4P_1x04_P5.08mm_Vertical
- moved J4 26.0 mm to (153.0, 122.6)
- moved J3 2.00 mm to (129.0, 122.6)
Connections:
- K3 pad 2: Net-(J3-Pin_6) -> Net-(J4-Pin_2)
- K3 pad 3: Net-(J3-Pin_5) -> Net-(J4-Pin_1)
- K4 pad 2: Net-(J3-Pin_8) -> Net-(J4-Pin_4)
- K4 pad 3: Net-(J3-Pin_7) -> Net-(J4-Pin_3)
- K5 pad 2: Net-(J4-Pin_2) -> Net-(J5-Pin_2)
- K5 pad 3: Net-(J4-Pin_1) -> Net-(J5-Pin_1)
- K6 pad 2: Net-(J4-Pin_4) -> Net-(J5-Pin_4)
- K6 pad 3: Net-(J4-Pin_3) -> Net-(J5-Pin_3)
- K7 pad 2: Net-(J4-Pin_6) -> Net-(J6-Pin_2)
- K7 pad 3: Net-(J4-Pin_5) -> Net-(J6-Pin_1)
- K8 pad 2: Net-(J4-Pin_8) -> Net-(J6-Pin_4)
- K8 pad 3: Net-(J4-Pin_7) -> Net-(J6-Pin_3)
- RV3 pad 1: Net-(J3-Pin_5) -> Net-(J4-Pin_1)
- RV3 pad 2: Net-(J3-Pin_6) -> Net-(J4-Pin_2)
- RV4 pad 1: Net-(J3-Pin_7) -> Net-(J4-Pin_3)
- RV4 pad 2: Net-(J3-Pin_8) -> Net-(J4-Pin_4)
- RV5 pad 1: Net-(J4-Pin_1) -> Net-(J5-Pin_1)
- RV5 pad 2: Net-(J4-Pin_2) -> Net-(J5-Pin_2)
- RV6 pad 1: Net-(J4-Pin_3) -> Net-(J5-Pin_3)
- RV6 pad 2: Net-(J4-Pin_4) -> Net-(J5-Pin_4)
- RV7 pad 1: Net-(J4-Pin_5) -> Net-(J6-Pin_1)
- RV7 pad 2: Net-(J4-Pin_6) -> Net-(J6-Pin_2)
- RV8 pad 1: Net-(J4-Pin_7) -> Net-(J6-Pin_3)
- RV8 pad 2: Net-(J4-Pin_8) -> Net-(J6-Pin_4)
Routing:
- net Net-(J4-Pin_8): track 66.6 -> 0.00 mm
- net Net-(J3-Pin_8): track 66.6 -> 0.00 mm
- net Net-(J6-Pin_4): track 0.00 -> 65.2 mm
- net Net-(J5-Pin_4): track 0.00 -> 65.2 mm
- net Net-(J3-Pin_6): track 65.1 -> 0.00 mm
- net Net-(J4-Pin_6): track 65.1 -> 0.00 mm
- net Net-(J6-Pin_2): track 0.00 -> 64.5 mm
- net Net-(J5-Pin_2): track 0.00 -> 64.5 mm
- net Net-(J4-Pin_7): track 49.7 -> 0.00 mm
- net Net-(J3-Pin_7): track 49.7 -> 0.00 mm
- net Net-(J6-Pin_3): track 0.00 -> 48.4 mm
- net Net-(J5-Pin_3): track 0.00 -> 48.4 mm
- net Net-(J4-Pin_5): track 48.2 -> 0.00 mm
- net Net-(J3-Pin_5): track 48.2 -> 0.00 mm
- net Net-(J6-Pin_1): track 0.00 -> 47.7 mm
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