File: V1/relay-24v-8ch-8a-v1.kicad_pcb (KiCad board)
At the start: 2 copper layers, 98 x 67.8 mm, 46 parts, among them J1 DB141V-2.54-6P, J2 DB141V-2.54-6P, J3 DB142V-5.08-4P, J4 DB142V-5.08-4P, J5 DB142V-5.08-4P, J6 DB142V-5.08-4P, K1 G5Q-1A4-DC24V, K2 G5Q-1A4-DC24V, K3 G5Q-1A4-DC24V, K4 G5Q-1A4-DC24V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

Commit message: Updated connectors
Parts:
- added J3: DB141V-2.54-4P, Tales:TerminalBlock_Dibo_DB141V-2.54-4P_1x04_P2.54mm_Vertical, F.Cu at (220.1, 67.9)
- J1: value DB141V-2.54-6P -> DB141V-2.54-2P; footprint Tales:TerminalBlock_Dibo_DB141V-2.54-6P_1x06_P2.54mm_Vertical -> Tales:TerminalBlock_Dibo_DB141V-2.54-2P_1x02_P2.54mm_Vertical
- J2: value DB141V-2.54-6P -> DB141V-2.54-4P; footprint Tales:TerminalBlock_Dibo_DB141V-2.54-6P_1x06_P2.54mm_Vertical -> Tales:TerminalBlock_Dibo_DB141V-2.54-4P_1x04_P2.54mm_Vertical
- R1, R2, R3, R4, R5, R6, R7, R8: value 5k6/100mW -> 6k8/100mW
- moved J2 47.9 mm to (172.1, 67.9)
- moved J1 34.5 mm to (206.5, 67.9)
- moved R5 3.00 mm to (196.3, 68.5)
- moved R6 3.00 mm to (196.3, 70.0)
- moved R7 3.00 mm to (196.3, 71.5)
- moved R8 3.00 mm to (196.3, 73.0)
- moved D11 2.00 mm to (181.3, 73.0)
- moved D13 2.00 mm to (186.3, 73.0)
- moved D15 2.00 mm to (191.3, 73.0)
- moved D9 2.00 mm to (176.3, 73.0)
- moved R1 1.00 mm to (150.3, 68.5)
- moved R2 1.00 mm to (150.3, 70.0)
- moved R3 1.00 mm to (150.3, 71.5)
- moved R4 1.00 mm to (150.3, 73.0)
- moved D10 0.50 mm to (178.2, 79.5)
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- renumbered J3 to J4, J4 to J5, J5 to J6, J6 to J7
Connections:
- J1 pad 1: Net-(D7-K) -> +24V
- J1 pad 2: Net-(D5-K) -> +24V
- J2 pad 1: Net-(D15-K) -> Net-(D7-K)
- J2 pad 2: Net-(D13-K) -> Net-(D5-K)
- J2 pad 3: Net-(D11-K) -> Net-(D3-K)
- J2 pad 4: Net-(D10-A) -> Net-(D1-K)
Routing:
- net +24V: track 250.9 -> 244.4 mm
- net Net-(J7-Pin_3): track 48.4 -> 45.8 mm
- net Net-(J7-Pin_1): track 47.7 -> 45.1 mm
- net Net-(J6-Pin_3): track 48.4 -> 45.8 mm
- net Net-(J6-Pin_1): track 47.7 -> 45.1 mm
- net Net-(J5-Pin_1): track 47.7 -> 45.1 mm
- net Net-(J4-Pin_3): track 48.4 -> 45.8 mm
- net Net-(J4-Pin_1): track 47.7 -> 45.1 mm
- net Net-(D13-K): track 45.3 -> 47.3 mm
- net Net-(D11-K): track 47.8 -> 49.8 mm
- net Net-(D15-K): track 47.1 -> 49.0 mm
- net Net-(D10-A): track 51.5 -> 52.7 mm
- net Net-(D9-A): track 21.3 -> 20.3 mm
- net Net-(D7-A): track 4.43 -> 3.43 mm
- net Net-(D5-A): track 10.0 -> 9.05 mm
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- added copper zone on B.Cu, net +24V
Other:
- board text removed: "IN6"

Commit message: Review before fabrication
Parts:
- R1, R2, R3, R4, R5, R6, R7, R8: value 6k8/100mW -> 10k/100mW
- moved K1 11.8 mm to (132.0, 93.8)
- moved K2 11.8 mm to (144.0, 93.8)
- moved K3 11.8 mm to (156.0, 93.8)
- moved K4 11.8 mm to (168.0, 93.8)
- moved K5 11.8 mm to (180.0, 93.8)
- moved K6 11.8 mm to (192.0, 93.8)
- moved K7 11.8 mm to (204.0, 93.8)
- moved K8 11.8 mm to (216.0, 93.8)
- moved J4 8.55 mm to (136.8, 119.0)
- moved J5 8.55 mm to (160.8, 119.0)
- moved J6 8.55 mm to (184.8, 119.0)
- moved J7 8.55 mm to (208.8, 119.0)
- moved J2 4.65 mm to (168.2, 70.5)
- moved J3 4.65 mm to (216.2, 70.5)
- moved RV1 3.58 mm to (132.0, 107.8)
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Connections:
- net Net-(D1-A) renamed /LED1
- net Net-(D1-K) renamed /IN1
- net Net-(D10-A) renamed /IN5
- net Net-(D11-A) renamed /LED6
- net Net-(D11-K) renamed /IN6
- net Net-(D13-A) renamed /LED7
- net Net-(D13-K) renamed /IN7
- net Net-(D15-A) renamed /LED8
- net Net-(D15-K) renamed /IN8
- net Net-(D3-A) renamed /LED2
- net Net-(D3-K) renamed /IN2
- net Net-(D5-A) renamed /LED3
- net Net-(D5-K) renamed /IN3
- net Net-(D7-A) renamed /LED4
- net Net-(D7-K) renamed /IN4
- net Net-(D9-A) renamed /LED5
- net Net-(J4-Pin_1) renamed /OUT1PW
- net Net-(J4-Pin_2) renamed /OUT1LD
- net Net-(J4-Pin_3) renamed /OUT2PW
- net Net-(J4-Pin_4) renamed /OUT2LD
- net Net-(J5-Pin_1) renamed /OUT3PW
- net Net-(J5-Pin_2) renamed /OUT3LD
- net Net-(J5-Pin_3) renamed /OUT4PW
- net Net-(J5-Pin_4) renamed /OUT4LD
- net Net-(J6-Pin_1) renamed /OUT5PW
- net Net-(J6-Pin_2) renamed /OUT5LD
- net Net-(J6-Pin_3) renamed /OUT6PW
- net Net-(J6-Pin_4) renamed /OUT6LD
- net Net-(J7-Pin_1) renamed /OUT7PW
- net Net-(J7-Pin_2) renamed /OUT7LD
- net Net-(J7-Pin_3) renamed /OUT8PW
- net Net-(J7-Pin_4) renamed /OUT8LD
Routing:
- net /IN5: track 52.7 -> 59.4 mm
- net /IN1: track 51.9 -> 58.5 mm
- net /IN7: track 47.3 -> 53.0 mm
- net /IN3: track 45.3 -> 51.0 mm
- net /IN2: track 47.8 -> 53.4 mm
- net /IN6: track 49.8 -> 55.4 mm
- net /OUT4PW: track 48.4 -> 43.2 mm
- net /IN8: track 49.0 -> 53.5 mm
- net /IN4: track 47.0 -> 51.4 mm
- net /OUT7LD: track 64.5 -> 61.1 mm
- net /OUT5LD: track 64.5 -> 61.1 mm
- net /OUT3LD: track 64.5 -> 61.1 mm
- net /OUT1LD: track 64.5 -> 61.1 mm
- net /OUT7PW: track 45.1 -> 41.7 mm
- net /OUT5PW: track 45.1 -> 41.7 mm
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- added copper zone on F.Cu, net +24V
- removed copper zone on B.Cu, net +24V
Other:
- rule pad_to_mask_clearance: 0 -> 0.1
